File: smarc_pcie_offboard_power/Power_Sequence.kicad_sch (KiCad schematic)
At the start: 31 parts, among them U1 TPS3808G50, U2 74LVC1G08, U4 TPS22992, U5 TPS22992, U6 TPS22992, U7 TPS22992

Commit message: power supply validated by codex
Parts:
- added D7, D8, D9: SCS521S-TG_30V, symbol Device:D_Zener_Small
- added J6: PH_2.0mm, symbol Connector:Conn_01x02_Pin
- added PC78, PC80, PC83: 0.1uF_10V, symbol Device:C_Small
- added PC79: 1nF_10V, symbol Device:C_Small
- added RP10: 0ohm_+-1%, symbol Device:R_Small_US
- added RP11, RP14: 100K_+-1%, symbol Device:R_Small_US
- added RP12: 106K_+-0.1%, symbol Device:R_Small_US
- added RP13: 9.88K_+-0.1%, symbol Device:R_Small_US
- added TP1: TestPoint, symbol Connector:TestPoint
- added U15: SN74LV1T08, symbol 74xGxx:74LVC1G08
- added U16: 74AHC1G09_SC70-5, symbol 74xGxx:74LVC1G08
- PC53, PC59, PC63, PC67: value 4.7nF_10V -> 4.7nF_50V
- U1: value TPS3808G50 -> TPS3808G01
- U4, U5, U6, U7: value TPS22992 -> TPS22992S
Connections:
- net P_+5V_A is gone; now on net P_+5V_ATX: PC60.2, PC61.1, RP3.2, RP7.2, RP8.2, RP9.2, U6.1 (VBIAS), U6.2 (VIN)
- net GND: now also PC47.1, PC78.1, PC79.2, PC80.2, PC83.1, RP11.2, RP13.2, U15.3 (GND), U16.3 (GND); no longer PC47.2
- net P_+1V8_S_PG: now also D9.1 (K)
- net P_+3V3_ATX: now also PC78.2, RP10.1, U15.5 (VCC)
- net P_+3V3_S_PG: now also D8.1 (K)
- net P_+5V_ATX: now also PC47.2, PC83.2, RP12.1, RP14.1, U16.5 (VCC); no longer PC47.1, U1.5 (SENSE)
- net P_+5V_S_PG: now also D7.1 (K)
- net at U1.3 (~{MR}): now also TP1.1
- net at U1.4 (CT): now also PC80.1, RP14.2
- net P_+3V3_5V_A_PG renamed S_CB_PWR_ON
- net S_CB_PWR_ON: now also RP10.2, RP11.1, U15.4
- net VIN_PWR_BAD#: no longer names the net of RP6.2
- net VIN_PWR_BAD#: now also J6.2 (Pin_2), U16.1; no longer U1.1 (~{RESET})
- new net: D7.2 (A), D8.2 (A), D9.2 (A), J6.1 (Pin_1)
- new net: PC79.1, RP12.2, RP13.1, U1.5 (SENSE)
- new net 5V_OK_N: U1.1 (~{RESET})
- new net CB_PWR_ON: U15.1
- new net CB_RESET_IN#: U16.4
- new net P_+3V3_5V_ATX_PG: U15.2
- new net RESET_IN#: U16.2
- no-connect marks 2 -> 0
Other:
- moved on the sheet: PC54, RP4, RP5, U2
