File: smarc_pcie_offboard_power/Power_Supply.kicad_sch (KiCad schematic)
At the start: 36 parts, among them J2 ATX-24, U3 TPS6282618

Commit message: power supply validated by codex
Parts:
- removed PC28, PC29, PC30, PC38, PC39, PC40: 22uF_6.3V, symbol Device:C_Small
- removed PQ1: 2N3904, Package_TO_SOT_THT:TO-92_Inline, symbol Transistor_BJT:2N3904
- removed PTC23, PTC24, PTC25: 150uF_6.3V, symbol Device:C_Small_US
- removed RP1: 4.7K_+-1%, symbol Device:R_Small_US
- L1: value 0.47uH_3A -> 0.47uH_5A
Connections:
- net P_+5V_A is gone; now on net P_+5V_ATX: J2.21 (+5V), J2.22 (+5V), J2.23 (+5V), J2.4 (+5V), J2.6 (+5V), PC31.1, PC35.1, PC36.1, PC44.1, PC45.1, PC46.1, PC50.1, PTC26.1, PTC29.1, PTC30.1, RP2.2, U3.6 (VIN)
- net GND: now also J2.16 (PS_ON#)
- net P_+5V_ATX: no longer J2.9 (+5VSB)
- net S_CB_PWR_ON: now also U3.1 (EN)
- net P_+3V3_5V_A_PG renamed P_+3V3_5V_ATX_PG
- net P_+3V3_5V_ATX_PG: no longer U3.1 (EN)
- no-connect marks 2 -> 3
Other:
- moved on the sheet: PC31, PC35, PC36, PC44, PC45, PC46, PTC26, PTC29, PTC30
