File: smarc_pcie_offboard_power/SMARC_CONNECTOR.kicad_sch (KiCad schematic)
At the start: 6 parts, among them J4 125B-78C00

Commit message: power supply validated by codex
Parts:
- removed F1: 5A_fuse, symbol Device:Fuse
- removed J4: 125B-78C00, symbol diode:125B-78C00
- removed PC37, PC38: 22uF_10V, symbol Device:C_Small
- removed PC39: 0.1uF_10V, symbol Device:C_Small
- removed RP15: 0ohm, symbol Device:R_Small_US
- added J4: 125B-78C00, symbol diode:125B-78C00
Connections:
- new net CAM_MCK: J4.S6 (CAM_MCK)
- new net CSI0_CK_N: J4.S9 (CSI0_CK-)
- new net CSI0_CK_P: J4.S8 (CSI0_CK+)
- new net CSI0_RX0_N: J4.S12 (CSI0_RX0-)
- new net CSI0_RX0_P: J4.S11 (CSI0_RX0+)
- new net CSI0_RX1_N: J4.S15 (CSI0_RX1-)
- new net CSI0_RX1_P: J4.S14 (CSI0_RX1+)
- new net CSI0_TX_I2C_CAM0_N: J4.S7 (CSI0_TX-/I2C_CAM0_DAT)
- new net CSI0_TX_I2C_CAM0_P: J4.S5 (CSI0_TX+/I2C_CAM0_CK)
- new net CSI1_CK_N: J4.P4 (CSI1_CK-)
- new net CSI1_CK_P: J4.P3 (CSI1_CK+)
- new net CSI1_RX0_N: J4.P8 (CSI1_RX0-)
- new net CSI1_RX0_P: J4.P7 (CSI1_RX0+)
- new net CSI1_RX1_N: J4.P11 (CSI1_RX1-)
- new net CSI1_RX1_P: J4.P10 (CSI1_RX1+)
- new net CSI1_RX2_N: J4.P14 (CSI1_RX2-)
- new net CSI1_RX2_P: J4.P13 (CSI1_RX2+)
- new net CSI1_RX3_N: J4.P17 (CSI1_RX3-)
- new net CSI1_RX3_P: J4.P16 (CSI1_RX3+)
- new net CSI1_TX_I2C_CAM1_N: J4.S2 (CSI1_TX-/I2C_CAM1_DAT)
- new net CSI1_TX_I2C_CAM1_P: J4.S1 (CSI1_TX+/I2C_CAM1_CK)
- new net DP1_AUX_HDMI_CTRL_N: J4.P106 (HDMI_CTRL_DAT/DP1_AUX-)
- new net DP1_AUX_HDMI_CTRL_P: J4.P105 (HDMI_CTRL_CK/DP1_AUX+)
- new net DP1_AUX_SEL: J4.P107 (DP1_AUX_SEL)
- new net DP1_LANE0_HDMI_D2_N: J4.P93 (HDMI_D2-/DP1_LANE0-)
- new net DP1_LANE0_HDMI_D2_P: J4.P92 (HDMI_D2+/DP1_LANE0+)
- new net DP1_LANE1_HDMI_D1_N: J4.P96 (HDMI_D1-/DP1_LANE1-)
- new net DP1_LANE1_HDMI_D1_P: J4.P95 (HDMI_D1+/DP1_LANE1+)
- new net DP1_LANE2_HDMI_D0_N: J4.P99 (HDMI_D0-/DP1_LANE2-)
- new net DP1_LANE2_HDMI_D0_P: J4.P98 (HDMI_D0+/DP1_LANE2+)
- new net DP1_LANE3_HDMI_CK_N: J4.P102 (HDMI_CK-/DP1_LANE3-)
- new net DP1_LANE3_HDMI_CK_P: J4.P101 (HDMI_CK+/DP1_LANE3+)
- new net HDMI_HPD_OR_DP1_HPD: J4.P104 (HDMI_HPD/DP1_HPD)
- no-connect marks 0 -> 2
Other:
- removed sheet Display Port
- removed sheet GPIO
- removed sheet Power Sequence
- removed sheet Power Supply
- removed sheet Smarc Connector
- removed sheet Switches and Reset
- removed sheet USB 3.0
- removed sheet USB 3.0 Power
- removed sheet uSD-CARD
- removed sheet x16 Card Slot
